File: USBPowerSupplyEurorack/_autosave-USBPowerSupplyEurorack.sch (KiCad schematic (older format))
At the start: 9 parts, among them J1 1734366-1, T1 RS6-0512D

Commit message: changed diode for lower forward voltage, prepared 2HP PCB contour
Parts:
- removed D1: SS36, SS36:DIOM8059X265N, symbol SS36:SS36
- added C3: 100nF close to Switch, symbol Device:CP_Small
- added D1: LSM115JE3_TR13, DIOM5436X330N, symbol LSM115JE3_TR13:LSM115JE3_TR13
- gave numbers to parts that had none: 3
Connections:
- no-connect marks 5 -> 4
Changed lines of the file:
@@
 $EndDescr
-$Comp
-L SS36:SS36 D1
-U 1 1 5FE03083
-P 2330 1470
-F 0 "D1" H 2730 1203 50  0000 C CNN
-F 1 "SS36" H 2730 1294 50  0000 C CNN
-F 2 "SS36:DIOM8059X265N" H 2830 1620 50  0001 L CNN
-F 3 "http://www.onsemi.com/pub/Collateral/SS39-D.PDF" H 2830 1520 50  0001 L CNN
-F 4 "ON SEMICONDUCTOR - SS36 - DIODE, SCHOTTKY, 3A, 60V, DO-214AB-3" H 2830 1420 50  0001 L CNN "Description"
-F 5 "2.65" H 2830 1320 50  0001 L CNN "Height"
-F 6 "ON Semiconductor" H 2830 1220 50  0001 L CNN "Manufacturer_Name"
-F 7 "SS36" H 2830 1120 50  0001 L CNN "Manufacturer_Part_Number"
-F 8 "SS36" H 2830 1020 50  0001 L CNN "Arrow Part Number"
-F 9 "https://www.arrow.com/en/products/ss36/on-semiconductor" H 2830 920 50  0001 L CNN "Arrow Price/Stock"
-F 10 "512-SS36" H 2830 820 50  0001 L CNN "Mouser Part Number"
-F 11 "https://www.mouser.co.uk/ProductDetail/ON-Semiconductor-Fairchild/SS36/?qs=3wuez3jz59JyNj1can%252BtMw%3D%3D" H 2830 720 50  0001 L CNN "Mouser Price/Stock"
-	1    2330 1470
-	-1   0    0    1
-$EndComp
 $Comp
 L Device:CP1_Small C1
@@
 +Vout
 $Comp
-L power:GND #PWR?
+L power:GND #PWR0101
 U 1 1 5FE13FD5
 P 1630 2110
-F 0 "#PWR?" H 1630 1860 50  0001 C CNN
+F 0 "#PWR0101" H 1630 1860 50  0001 C CNN
 F 1 "GND" H 1635 1937 50  0000 C CNN
 F 2 "" H 1630 2110 50  0001 C CNN
@@
 Connection ~ 4430 1870
 $Comp
-L power:+5VD #PWR?
+L power:+5VD #PWR0102
 U 1 1 5FE20BD7
 P 2310 1420
-F 0 "#PWR?" H 2310 1270 50  0001 C CNN
+F 0 "#PWR0102" H 2310 1270 50  0001 C CNN
 F 1 "+5VD" H 2325 1593 50  0000 C CNN
 F 2 "" H 2310 1420 50  0001 C CNN
@@
 $EndComp
 $Comp
-L power:+5V #PWR?
+L power:+5V #PWR0103
 U 1 1 5FE2195B
 P 4430 1370
-F 0 "#PWR?" H 4430 1220 50  0001 C CNN
+F 0 "#PWR0103" H 4430 1220 50  0001 C CNN
 F 1 "+5V" H 4445 1543 50  0000 C CNN
 F 2 "" H 4430 1370 50  0001 C CNN
@@
 Connection ~ 4430 1370
 $Comp
-L power:+5VD #PWR?
+L power:+5VD #PWR0104
 U 1 1 5FE220CC
 P 3030 1870
-F 0 "#PWR?" H 3030 1720 50  0001 C CNN
+F 0 "#PWR0104" H 3030 1720 50  0001 C CNN
 F 1 "+5VD" H 3045 2043 50  0000 C CNN
 F 2 "" H 3030 1870 50  0001 C CNN
@@
 Connection ~ 3030 1870
 $Comp
-L Device:R_Small R?
+L Device:R_Small R1
 U 1 1 5FE234A2
 P 3730 2670
-F 0 "R?" H 3789 2716 50  0000 L CNN
+F 0 "R1" H 3789 2716 50  0000 L CNN
 F 1 "100" H 3789 2625 50  0000 L CNN
 F 2 "" H 3730 2670 50  0001 C CNN
@@
 $EndComp
 $Comp
-L power:GND #PWR?
+L power:GND #PWR0105
 U 1 1 5FE23B35
 P 3730 2820
-F 0 "#PWR?" H 3730 2570 50  0001 C CNN
+F 0 "#PWR0105" H 3730 2570 50  0001 C CNN
 F 1 "GND" H 3735 2647 50  0000 C CNN
 F 2 "" H 3730 2820 50  0001 C CNN
@@
 Push button & LED
 $Comp
-L power:+5V #PWR?
+L power:+5V #PWR0106
 U 1 1 5FE2FAE8
 P 5630 4740
-F 0 "#PWR?" H 5630 4590 50  0001 C CNN
+F 0 "#PWR0106" H 5630 4590 50  0001 C CNN
 F 1 "+5V" H 5645 4913 50  0000 C CNN
 F 2 "" H 5630 4740 50  0001 C CNN
@@
 NoConn ~ 1510 1670
 $Comp
-L 744235601:744235601 L?
+L Device:CP1_Small C2
+U 1 1 5FE2664F
+P 6420 5130
+F 0 "C2" H 6511 5176 50  0000 L CNN
+F 1 "22uF" H 6511 5085 50  0000 L CNN
+F 2 "" H 6420 5130 50  0001 C CNN
+F 3 "~" H 6420 5130 50  0001 C CNN
+	1    6420 5130
+	1    0    0    -1
+$EndComp
+Wire Wire Line
+	6420 5230 6420 5420
+Wire Wire Line
+	6420 5030 6420 4840
+Wire Wire Line
+	6010 4970 6010 4840
+Wire Wire Line
+	6010 4840 6420 4840
+Connection ~ 6420 4840
+Wire Wire Line
+	6010 5270 6010 5420
+Wire Wire Line
+	6010 5420 6420 5420
+Connection ~ 6420 5420
+Wire Wire Line
+	5630 5020 5630 4840
+Wire Wire Line
+	5630 4840 6010 4840
+Connection ~ 6010 4840
+Wire Wire Line
+	5630 5220 5630 5420
+Wire Wire Line
+	5630 5420 6010 5420
+Connection ~ 6010 5420
+$Comp
+L power:GND #PWR0107
+U 1 1 5FE34916
+P 5630 5520
+F 0 "#PWR0107" H 5630 5270 50  0001 C CNN
+F 1 "GND" H 5635 5347 50  0000 C CNN
+F 2 "" H 5630 5520 50  0001 C CNN
+F 3 "" H 5630 5520 50  0001 C CNN
+	1    5630 5520
+	1    0    0    -1
+$EndComp
+Wire Wire Line
+	5630 5520 5630 5420
+Connection ~ 5630 5420
+Wire Wire Line
+	2230 1470 2310 1470
+Wire Wire Line
+	2310 1470 2310 1420
+Wire Wire Line
+	5630 4740 5630 4840
+Connection ~ 5630 4840
+Text GLabel 9120 4870 2    50   Input ~ 0
++Vin
+Text GLabel 9400 5180 2    50   Input ~ 0
+-Vin
+Wire Wire Line
+	6830 4840 6830 5090
+Wire Wire Line
+	6420 4840 6830 4840
+Wire Wire Line
+	6830 5420 6830 5190
+Wire Wire Line
+	6420 5420 6830 5420
+$Comp
+L 744235601:744235601 L1
 U 1 1 5FE25D51
 P 6830 5090
-F 0 "L?" H 7230 5355 50  0000 C CNN
+F 0 "L1" H 7230 5355 50  0000 C CNN
 F 1 "744235601" H 7230 5264 50  0000 C CNN
 F 2 "744235601" H 7480 5190 50  0001 L CNN
@@
 $EndComp
 $Comp
-L Device:CP1_Small C?
-U 1 1 5FE2664F
-P 6420 5130
-F 0 "C?" H 6511 5176 50  0000 L CNN
-F 1 "22uF" H 6511 5085 50  0000 L CNN
-F 2 "" H 6420 5130 50  0001 C CNN
-F 3 "~" H 6420 5130 50  0001 C CNN
-	1    6420 5130
-	1    0    0    -1
-$EndComp
-Wire Wire Line
-	6420 5230 6420 5420
-Wire Wire Line
-	6420 5420 6830 5420
-Wire Wire Line
-	6830 5420 6830 5190
-Wire Wire Line
-	6420 5030 6420 4840
-Wire Wire Line
-	6420 4840 6830 4840
-Wire Wire Line
-	6830 4840 6830 5090
-Wire Wire Line
-	6010 4970 6010 4840
-Wire Wire Line
-	6010 4840 6420 4840
-Connection ~ 6420 4840
-Wire Wire Line
-	6010 5270 6010 5420
-Wire Wire Line
-	6010 5420 6420 5420
-Connection ~ 6420 5420
-Wire Wire Line
-	5630 5020 5630 4840
-Wire Wire Line
-	5630 4840 6010 4840
-Connection ~ 6010 4840
-Wire Wire Line
-	5630 5220 5630 5420
-Wire Wire Line
-	5630 5420 6010 5420
-Connection ~ 6010 5420
-$Comp
-L power:GND #PWR?
-U 1 1 5FE34916
-P 5630 5520
-F 0 "#PWR?" H 5630 5270 50  0001 C CNN
-F 1 "GND" H 5635 5347 50  0000 C CNN
-F 2 "" H 5630 5520 50  0001 C CNN
-F 3 "" H 5630 5520 50  0001 C CNN
-	1    5630 5520
-	1    0    0    -1
-$EndComp
-Wire Wire Line
-	5630 5520 5630 5420
-Connection ~ 5630 5420
-Text GLabel 7630 5190 2    50   Input ~ 0
--Vin
-Text GLabel 7630 5090 2    50   Input ~ 0
-+Vin
-Wire Wire Line
-	2230 1470 2310 1470
-Wire Wire Line
-	2310 1470 2310 1420
-Wire Wire Line
-	5630 4740 5630 4840
-Connection ~ 5630 4840
-NoConn ~ 7140 2870
+L Device:CP_Small C3
+U 1 1 5FE49BEB
+P 8000 5130
+F 0 "C3" H 8088 5176 50  0000 L CNN
+F 1 "100nF close to Switch" H 8088 5085 50  0000 L CNN
+F 2 "" H 8000 5130 50  0001 C CNN
+F 3 "~" H 8000 5130 50  0001 C CNN
+	1    8000 5130
+	1    0    0    -1
+$EndComp
+$Comp
+L LSM115JE3_TR13:LSM115JE3_TR13 D1
+U 1 1 5FE4DB5C
+P 2330 1470
+F 0 "D1" H 2800 1230 50  0000 C CNN
+F 1 "LSM115JE3_TR13" H 2810 1310 50  0000 C CNN
+F 2 "DIOM5436X330N" H 2830 1620 50  0001 L CNN
+F 3 "https://media.digikey.com/pdf/Data%20Sheets/Microsemi%20PDFs/LSM115J.pdf" H 2830 1520 50  0001 L CNN
+F 4 "Schottky Diodes & Rectifiers Schottky" H 2830 1420 50  0001 L CNN "Description"
+F 5 "3.3" H 2830 1320 50  0001 L CNN "Height"
+F 6 "Microsemi Corporation" H 2830 1220 50  0001 L CNN "Manufacturer_Name"
+F 7 "LSM115JE3/TR13" H 2830 1120 50  0001 L CNN "Manufacturer_Part_Number"
+F 8 "LSM115JE3/TR13" H 2830 1020 50  0001 L CNN "Arrow Part Number"
+F 9 "https://www.arrow.com/en/products/lsm115je3tr13/microsemi" H 2830 920 50  0001 L CNN "Arrow Price/Stock"
+F 10 "494-LSM115JE3/TR13" H 2830 820 50  0001 L CNN "Mouser Part Number"
+F 11 "https://www.mouser.co.uk/ProductDetail/Microchip-Microsemi/LSM115JE3-TR13?qs=6jAvgNDGUA8H9k1qUsKdHA%3D%3D" H 2830 720 50  0001 L CNN "Mouser Price/Stock"
+	1    2330 1470
+	-1   0    0    1
+$EndComp
 $EndSCHEMATC
