File: USBPowerSupplyEurorack/_autosave-USBPowerSupplyEurorack.sch (KiCad schematic (older format))
At the start: 21 parts, among them J1 1734366-1, J2 95278-501A10LF, Q1 Q_PMOS_GSD

Commit message: changed footprints placement, added the two LEDs
Parts:
- D2, D5: renamed from D?; footprint (none) -> digikey-footprints:LED_0603
- gave numbers to parts that had none: 1
Changed lines of the file:
@@
 Connection ~ 4915 5905
 $Comp
-L Device:LED_Small_ALT D?
+L Device:LED_Small_ALT D2
 U 1 1 5FF1E6C4
 P 3075 5330
-F 0 "D?" V 3121 5260 50  0000 R CNN
+F 0 "D2" V 3121 5260 50  0000 R CNN
 F 1 "Blue" V 3030 5260 50  0000 R CNN
-F 2 "" V 3075 5330 50  0001 C CNN
+F 2 "digikey-footprints:LED_0603" V 3075 5330 50  0001 C CNN
 F 3 "~" V 3075 5330 50  0001 C CNN
 	1    3075 5330
@@
 	3075 5165 3450 5165
 $Comp
-L Device:R_Small R?
+L Device:R_Small R2
 U 1 1 5FF3D1E7
 P 3075 6120
-F 0 "R?" H 3134 6166 50  0000 L CNN
+F 0 "R2" H 3134 6166 50  0000 L CNN
 F 1 "1K" H 3134 6075 50  0000 L CNN
 F 2 "Resistor_SMD:R_0805_2012Metric" H 3075 6120 50  0001 C CNN
@@
 $EndComp
 $Comp
-L Device:LED_Small_ALT D?
+L Device:LED_Small_ALT D5
 U 1 1 5FF3D1ED
 P 3075 5920
-F 0 "D?" V 3121 5850 50  0000 R CNN
+F 0 "D5" V 3121 5850 50  0000 R CNN
 F 1 "Blue" V 3030 5850 50  0000 R CNN
-F 2 "" V 3075 5920 50  0001 C CNN
+F 2 "digikey-footprints:LED_0603" V 3075 5920 50  0001 C CNN
 F 3 "~" V 3075 5920 50  0001 C CNN
 	1    3075 5920
